File: Flashlight.kicad_pcb (KiCad board)
At the start: 2 copper layers, 99.4 x 99.4 mm, 10 parts

Commit message: Finalized Kicad PCB Design
Parts:
- moved D1 0.10 mm to (150.0, 79.9)
Connections:
- D1 pad 2: /5V -> /12V1
- D10 pad 2: /5V -> /12V3
- D2 pad 2: /5V -> /12V2
- D3 pad 2: /5V -> /12V2
- D4 pad 2: /5V -> /12V2
- D5 pad 2: /5V -> /12V2
- D6 pad 2: /5V -> /12V2
- D7 pad 2: /5V -> /12V3
- D8 pad 2: /5V -> /12V3
- D9 pad 2: /5V -> /12V3
Routing:
- net /5V: vias 96 -> 0
- net /12V3: vias 0 -> 48
- net /12V2: vias 0 -> 48
- net /12V1: vias 0 -> 24
- added copper zone on B.Cu, net /12V1
- added copper zone on F.Cu, net /12V1
- added copper zone on B.Cu, net /12V2
- added copper zone on F.Cu, net /12V2
- added copper zone on B.Cu, net /12V3
- added copper zone on F.Cu, net /12V3
- removed copper zone on B.Cu, net /5V
- removed copper zone on F.Cu, net /5V
Other:
- outline, holes or cut-outs redrawn
- board text added: "K"

Commit message: Changed some PCB things
Other:
- outline, holes or cut-outs redrawn
